File: Tuner/TandemMatch/TandemMatch.sch (KiCad schematic (older format))
At the start: 69 parts, among them J1 Conn_01x02, J10 Conn_01x01, J11 Conn_01x01, J12 Conn_01x01, J13 Conn_01x01, J14 Conn_01x01, J15 Conn_01x01, J16 Conn_01x01, J17 Barrel_Jack, J18 Conn_Coaxial, J19 Conn_01x02, J2 Conn_01x02, J20 Conn_Coaxial, J21 Conn_01x01, J22 Conn_01x01, J23 Conn_01x01, J24 Conn_01x01, J25 Conn_01x01, J26 Conn_01x01, J27 Conn_01x01, J28 Conn_01x01, J29 Conn_01x01, J3 Conn_Coaxial, J30 Conn_01x01, J31 Conn_01x01, J32 Conn_01x01, J33 Conn_01x03, J4 Conn_Coaxial, J5 Conn_01x01, J6 Conn_01x01, J7 Conn_01x01, J8 Conn_01x01, J9 Conn_01x01

Commit message: Actually tuning code now!
Parts:
- added JP7, JP8: Jumper_NC_Small, Pin_Headers:Pin_Header_Straight_1x02_Pitch2.54mm, symbol Jumper_NC_Small
Connections:
- net at J7.1 (Pin_1), JP5.2, JP9.2: now also JP7.1; no longer J3.1 (In)
- net at J11.1 (Pin_1), J31.1 (Pin_1), JP12.2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: now also JP8.2; no longer J18.1 (In)
- new net: J3.1 (In), JP7.2
- new net: J18.1 (In), JP8.1
Other:
- moved on the sheet: JP12
Changed lines of the file:
@@
 L Jumper_NC_Small JP12
 U 1 1 5C77AC18
-P 5400 2250
-F 0 "JP12" H 5400 2330 50  0000 C CNN
-F 1 "Jumper_NC_Small" H 5410 2190 50  0000 C CNN
-F 2 "Pin_Headers:Pin_Header_Straight_1x02_Pitch2.54mm" H 5400 2250 50  0001 C CNN
-F 3 "" H 5400 2250 50  0001 C CNN
-	1    5400 2250
+P 5300 2250
+F 0 "JP12" H 5300 2330 50  0000 C CNN
+F 1 "Jumper_NC_Small" H 5310 2190 50  0000 C CNN
+F 2 "Pin_Headers:Pin_Header_Straight_1x02_Pitch2.54mm" H 5300 2250 50  0001 C CNN
+F 3 "" H 5300 2250 50  0001 C CNN
+	1    5300 2250
 	0    1    1    0
 $EndComp
@@
 $EndComp
 Wire Wire Line
-	4250 2800 5600 2800
+	4250 2800 5350 2800
 Wire Wire Line
 	2400 3600 2400 3400
-Wire Wire Line
-	2050 2800 2950 2800
 Wire Wire Line
 	5050 3700 5050 3500
@@
 Wire Wire Line
 	2450 2550 2450 2800
-Connection ~ 2450 2800
 Wire Wire Line
 	5050 2350 5050 2100
@@
 	2400 6450 2400 6400
 Wire Wire Line
-	2700 2550 2700 2800
+	2700 2800 2700 2550
 Connection ~ 2700 2800
-Connection ~ 5400 2800
-Wire Wire Line
-	5650 1250 5400 1250
-Wire Wire Line
-	5400 2350 5400 2800
-Wire Wire Line
-	5400 1250 5400 2150
+Wire Wire Line
+	5300 1250 5650 1250
 Wire Wire Line
 	5450 4650 5450 4950
@@
 Connection ~ 10250 2600
 Connection ~ 10250 2300
+Wire Wire Line
+	2350 2800 2950 2800
+$Comp
+L Jumper_NC_Small JP7
+U 1 1 5C82E8F5
+P 2250 2800
+F 0 "JP7" H 2250 2880 50  0000 C CNN
+F 1 "Jumper_NC_Small" H 2260 2740 50  0000 C CNN
+F 2 "Pin_Headers:Pin_Header_Straight_1x02_Pitch2.54mm" H 2250 2800 50  0001 C CNN
+F 3 "" H 2250 2800 50  0001 C CNN
+	1    2250 2800
+	-1   0    0    1
+$EndComp
+Connection ~ 2450 2800
+Wire Wire Line
+	2150 2800 2050 2800
+Wire Wire Line
+	5300 2800 5300 2350
+Wire Wire Line
+	5300 2150 5300 1250
+$Comp
+L Jumper_NC_Small JP8
+U 1 1 5C82F0DD
+P 5450 2800
+F 0 "JP8" H 5450 2880 50  0000 C CNN
+F 1 "Jumper_NC_Small" H 5460 2740 50  0000 C CNN
+F 2 "Pin_Headers:Pin_Header_Straight_1x02_Pitch2.54mm" H 5450 2800 50  0001 C CNN
+F 3 "" H 5450 2800 50  0001 C CNN
+	1    5450 2800
+	-1   0    0    1
+$EndComp
+Wire Wire Line
+	5600 2800 5550 2800
+Connection ~ 5300 2800
 $EndSCHEMATC
