File: Tuner/Controller/ControllerPhase.sch (KiCad schematic (older format))
At the start: 79 parts, among them Q1 2N3904, Q3 2N3904, Q4 2N3904, Q5 2N3904, Q6 2N3904, Q7 2N3904, Q8 2N3904, U1 74LS393, U2 74HC14, U3 74HC86

Commit message: A few tweaks
Parts:
- added C43, C44, C45: 10 nF, Capacitors_THT:C_Disc_D5.0mm_W2.5mm_P2.50mm, symbol C
Connections:
- net XCur: now also C44.2; no longer R22.1
- net XFwd: now also C45.2; no longer R41.1
- net XRev: now also C43.2; no longer R28.1
- new net: C43.1, R28.1
- new net: C44.1, R22.1
- new net: C45.1, R41.1
Changed lines of the file:
@@
 Text GLabel 7400 2650 2    60   Input ~ 0
 PhaseFwd
-Text GLabel 1150 5600 1    60   Input ~ 0
+Text GLabel 1150 5100 1    60   Input ~ 0
 XFwd
 $Comp
@@
 	0    -1   1    0
 $EndComp
-Text GLabel 1100 1400 1    60   Input ~ 0
+Text GLabel 1100 950  1    60   Input ~ 0
 XRev
 Text GLabel 3350 2150 3    60   Input ~ 0
@@
 	-1   0    0    -1
 $EndComp
-Text GLabel 1100 3250 1    60   Input ~ 0
+Text GLabel 1100 2950 1    60   Input ~ 0
 XCur
 Text GLabel 3350 4000 3    60   Input ~ 0
@@
 	2500 5450 2150 5450
 Wire Wire Line
-	2700 6050 2700 5800
+	2700 5800 2700 6050
 Wire Wire Line
 	2700 5850 2750 5850
@@
 	2450 1250 2100 1250
 Wire Wire Line
-	2650 1850 2650 1600
+	2650 1600 2650 1850
 Wire Wire Line
 	2650 1650 2700 1650
@@
 	2450 3150 2100 3150
 Wire Wire Line
-	2650 3750 2650 3500
+	2650 3500 2650 3750
 Wire Wire Line
 	2650 3550 2700 3550
@@
 	1350 1550 1650 1550
 Wire Wire Line
-	1100 1400 1100 1600
+	1100 1300 1100 1600
 $Comp
 L R R22
@@
 Connection ~ 1350 3850
 Wire Wire Line
-	1100 3250 1100 3500
-Wire Wire Line
 	1350 3450 1650 3450
 Wire Wire Line
@@
 Wire Wire Line
 	1700 5750 1700 5800
-Wire Wire Line
-	1150 5800 1150 5600
 $Comp
 L R R50
@@
 Wire Wire Line
 	2950 2000 2800 2000
+$Comp
+L C C43
+U 1 1 5C81FCDA
+P 1100 1150
+F 0 "C43" H 1125 1250 50  0000 L CNN
+F 1 "10 nF" V 1050 1200 50  0000 L CNN
+F 2 "Capacitors_THT:C_Disc_D5.0mm_W2.5mm_P2.50mm" H 1138 1000 50  0001 C CNN
+F 3 "" H 1100 1150 50  0001 C CNN
+	1    1100 1150
+	-1   0    0    1
+$EndComp
+Wire Wire Line
+	1100 950  1100 1000
+$Comp
+L C C44
+U 1 1 5C82067D
+P 1100 3200
+F 0 "C44" H 1125 3300 50  0000 L CNN
+F 1 "10 nF" V 1050 3250 50  0000 L CNN
+F 2 "Capacitors_THT:C_Disc_D5.0mm_W2.5mm_P2.50mm" H 1138 3050 50  0001 C CNN
+F 3 "" H 1100 3200 50  0001 C CNN
+	1    1100 3200
+	-1   0    0    1
+$EndComp
+Wire Wire Line
+	1100 3050 1100 2950
+Wire Wire Line
+	1100 3350 1100 3500
+$Comp
+L C C45
+U 1 1 5C820F02
+P 1150 5450
+F 0 "C45" H 1175 5550 50  0000 L CNN
+F 1 "10 nF" V 1100 5500 50  0000 L CNN
+F 2 "Capacitors_THT:C_Disc_D5.0mm_W2.5mm_P2.50mm" H 1188 5300 50  0001 C CNN
+F 3 "" H 1150 5450 50  0001 C CNN
+	1    1150 5450
+	-1   0    0    1
+$EndComp
+Wire Wire Line
+	1150 5300 1150 5100
+Wire Wire Line
+	1150 5600 1150 5800
 $EndSCHEMATC
