File: Tuner/QuadCoupler/QuadCoupler.sch (KiCad schematic (older format))
At the start: 102 parts, among them J1 Conn_01x01, J10 Conn_01x02, J11 Conn_01x01, J12 Conn_01x01, J13 Conn_01x01, J14 Conn_01x01, J15 Conn_01x01, J17 Conn_01x01, J19 Conn_01x02, J2 Conn_Coaxial, J21 Conn_01x01, J22 Conn_01x01, J23 Conn_01x01, J24 Conn_01x01, J3 Conn_Coaxial, J4 Conn_Coaxial, J5 Conn_Coaxial, J6 Conn_Coaxial, J7 Conn_01x01, J8 Conn_01x01, J9 Conn_01x01

Commit message: A few tweaks
Parts:
- added C20, C21, C22, C23: NC, Capacitors_THT:C_Disc_D5.0mm_W2.5mm_P5.00mm, symbol C_Small
Connections:
- net at C13.2, C15.2, JP4.2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: now also C21.2
- net at C13.1, C17.2, JP6.2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: now also C20.2
- net at C12.2, C16.2, JP9.1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: now also C22.2
- net at C12.1, C18.2, JP5.1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: now also C23.2
- net at C17.1, J11.1 (Pin_1), J2.1 (In): now also C20.1
- net at C15.1, J17.1 (Pin_1), J4.1 (In): now also C21.1
- net at C18.1, J13.1 (Pin_1), J5.1 (In): now also C23.1
- net at C16.1, J15.1 (Pin_1), J6.1 (In): now also C22.1
Changed lines of the file:
@@
 	3100 5800 3100 5650
 Wire Wire Line
-	5550 5650 5550 5450
-Wire Wire Line
-	5550 5450 5850 5450
+	5550 5450 5550 5800
+Wire Wire Line
+	5850 5450 5550 5450
 Connection ~ 5550 5650
 Wire Wire Line
@@
 Connection ~ 4150 6600
 Wire Wire Line
-	5550 6600 5550 7150
+	5550 6450 5550 7150
 Wire Wire Line
 	5550 7150 6000 7150
@@
 	8100 2200 8100 2100
 Connection ~ 8100 2100
+$Comp
+L C_Small C20
+U 1 1 5C819FC4
+P 4700 1850
+F 0 "C20" H 4710 1920 50  0000 L CNN
+F 1 "NC" H 4710 1770 50  0000 L CNN
+F 2 "Capacitors_THT:C_Disc_D5.0mm_W2.5mm_P5.00mm" H 4700 1850 50  0001 C CNN
+F 3 "" H 4700 1850 50  0001 C CNN
+	1    4700 1850
+	0    1    1    0
+$EndComp
+Wire Wire Line
+	4500 1750 4500 1850
+Wire Wire Line
+	4500 1850 4600 1850
+Connection ~ 4500 1750
+Wire Wire Line
+	4900 1750 4900 1850
+Wire Wire Line
+	4900 1850 4800 1850
+Connection ~ 4900 1750
+$Comp
+L C_Small C21
+U 1 1 5C81A810
+P 5150 2500
+F 0 "C21" H 5160 2570 50  0000 L CNN
+F 1 "NC" H 5160 2420 50  0000 L CNN
+F 2 "Capacitors_THT:C_Disc_D5.0mm_W2.5mm_P5.00mm" H 5150 2500 50  0001 C CNN
+F 3 "" H 5150 2500 50  0001 C CNN
+	1    5150 2500
+	0    1    1    0
+$EndComp
+Wire Wire Line
+	5050 2500 4950 2500
+Wire Wire Line
+	4950 2500 4950 2700
+Connection ~ 4950 2700
+Wire Wire Line
+	5250 2500 5350 2500
+Wire Wire Line
+	5350 2500 5350 2700
+Connection ~ 5350 2700
+$Comp
+L C_Small C23
+U 1 1 5C81AF45
+P 5400 5800
+F 0 "C23" H 5410 5870 50  0000 L CNN
+F 1 "NC" H 5410 5720 50  0000 L CNN
+F 2 "Capacitors_THT:C_Disc_D5.0mm_W2.5mm_P5.00mm" H 5400 5800 50  0001 C CNN
+F 3 "" H 5400 5800 50  0001 C CNN
+	1    5400 5800
+	0    1    1    0
+$EndComp
+Wire Wire Line
+	5200 5650 5200 5800
+Wire Wire Line
+	5200 5800 5300 5800
+Connection ~ 5200 5650
+Wire Wire Line
+	5550 5800 5500 5800
+$Comp
+L C_Small C22
+U 1 1 5C81B552
+P 5350 6450
+F 0 "C22" H 5360 6520 50  0000 L CNN
+F 1 "NC" H 5360 6370 50  0000 L CNN
+F 2 "Capacitors_THT:C_Disc_D5.0mm_W2.5mm_P5.00mm" H 5350 6450 50  0001 C CNN
+F 3 "" H 5350 6450 50  0001 C CNN
+	1    5350 6450
+	0    1    1    0
+$EndComp
+Wire Wire Line
+	5450 6450 5550 6450
+Wire Wire Line
+	5250 6450 5150 6450
+Wire Wire Line
+	5150 6450 5150 6600
+Connection ~ 5150 6600
 $EndSCHEMATC

Commit message: JLCPCB order 2019-03-25
Parts:
- added C24, C25: NC, Capacitors_THT:C_Disc_D5.0mm_W2.5mm_P5.00mm, symbol C_Small
- added J16: Conn_01x01, Connectors:1pin, symbol Conn_01x01
Connections:
- net at C7.1, TR1.2 (P2): now also C24.1, C25.1; no longer J3.1 (In)
- new net: C24.2, C25.2, J16.1 (Pin_1), J3.1 (In)
Other:
- note added: "14:10 or 20:14 \nP3:P2 trifilar\nimpedance\nautotransformer"
- note removed: "9:4 P3:P2\ntrifilar\nimpedance\nautotransformer"
Changed lines of the file:
@@
 	1    0    0    -1
 $EndComp
-Text Notes 1650 3550 0    60   ~ 0
-9:4 P3:P2\ntrifilar\nimpedance\nautotransformer
 Text Notes 3100 3500 0    60   ~ 0
 1:1 bifilar\nautotransformer
@@
 $EndComp
 Text Notes 1700 1600 0    60   ~ 0
-9:4 P3:P2\ntrifilar\nimpedance\nautotransformer
+14:10 or 20:14 \nP3:P2 trifilar\nimpedance\nautotransformer
 Text Notes 2950 2100 0    60   ~ 0
 1:1 bifilar\nautotransformer
@@
 	1    0    0    -1
 $EndComp
-Text Notes 1650 5500 0    60   ~ 0
-9:4 P3:P2\ntrifilar\nimpedance\nautotransformer
 Text Notes 2900 6000 0    60   ~ 0
 1:1 bifilar\nautotransformer
@@
 	750  4150 750  4050
 Wire Wire Line
-	900  4150 1650 4150
-Wire Wire Line
-	900  3850 900  4150
+	900  3600 900  4150
 Connection ~ 7000 4050
 Connection ~ 7000 3750
@@
 	4200 2700 4200 2350
 Wire Wire Line
-	1250 4300 1250 4150
+	1250 4000 1250 4300
 Connection ~ 1250 4150
 Wire Wire Line
@@
 	5150 6450 5150 6600
 Connection ~ 5150 6600
+$Comp
+L C_Small C25
+U 1 1 5C977A27
+P 1050 4150
+F 0 "C25" H 1060 4220 50  0000 L CNN
+F 1 "NC" H 1060 4070 50  0000 L CNN
+F 2 "Capacitors_THT:C_Disc_D5.0mm_W2.5mm_P5.00mm" H 1050 4150 50  0001 C CNN
+F 3 "" H 1050 4150 50  0001 C CNN
+	1    1050 4150
+	0    1    1    0
+$EndComp
+Wire Wire Line
+	1150 4150 1650 4150
+Wire Wire Line
+	900  4150 950  4150
+$Comp
+L C_Small C24
+U 1 1 5C978024
+P 1050 4000
+F 0 "C24" H 1060 4070 50  0000 L CNN
+F 1 "NC" H 1060 3920 50  0000 L CNN
+F 2 "Capacitors_THT:C_Disc_D5.0mm_W2.5mm_P5.00mm" H 1050 4000 50  0001 C CNN
+F 3 "" H 1050 4000 50  0001 C CNN
+	1    1050 4000
+	0    1    1    0
+$EndComp
+Wire Wire Line
+	950  4000 900  4000
+Connection ~ 900  4000
+Wire Wire Line
+	1150 4000 1250 4000
+$Comp
+L Conn_01x01 J16
+U 1 1 5C9788D2
+P 1200 3600
+F 0 "J16" H 1200 3700 50  0000 C CNN
+F 1 "Conn_01x01" H 1200 3500 50  0000 C CNN
+F 2 "Connectors:1pin" H 1200 3600 50  0001 C CNN
+F 3 "" H 1200 3600 50  0001 C CNN
+	1    1200 3600
+	1    0    0    -1
+$EndComp
+Wire Wire Line
+	900  3600 1000 3600
+Connection ~ 900  3850
+Text Notes 1650 3550 0    60   ~ 0
+14:10 or 20:14 \nP3:P2 trifilar\nimpedance\nautotransformer
+Text Notes 1650 5550 0    60   ~ 0
+14:10 or 20:14 \nP3:P2 trifilar\nimpedance\nautotransformer
 $EndSCHEMATC
